File: pcb/extinction_button.kicad_sch (KiCad schematic)
At the start: 35 parts, among them J1 DX07S016JA1R1500, J2 Conn_01x02, J3 Conn_01x06, SW1 R-667843, U1 ATmega32U4-A, U2 MIC5219-5.0YM5, Y1 ECS-160-10-36-CKM-TR3

Commit message: add reverse mounted led
Parts:
- added LED4: 4960, 4960_ADA, symbol SK6812-E:4960
Connections:
- net D4: now also LED4.4 (DIN); no longer D7.4 (DIN)
- net GND: now also LED4.3 (GND)
- net VCC: now also LED4.1 (VDD)
- new net: D7.4 (DIN), LED4.2 (DOUT)
