File: pcb/one_button.kicad_sch (KiCad schematic)
At the start: 46 parts, among them J1 DX07S016JA1R1500, J2 Conn_01x02, J3 Conn_01x06, SW1 R-667843, U1 ATmega32U4-A, U2 MIC5219-5.0YM5, U3 1SS400T1G, Y1 ECS-160-10-36-CKM-TR3

Commit message: fix pcb, firmware
Parts:
- removed LED1, LED2: LTST-C191KSKT, footprints:LED_LTST-C191KRKT_LTO, symbol 2023-12-05_05-19-35:LTST-C191KSKT
- removed LED4: 4960, 4960_ADA, symbol SK6812-E:4960
- removed R4, R5: 330, Resistor_SMD:R_0805_2012Metric, symbol Device:R
Connections:
- net D4: now also D7.4 (DIN)
- no-connect marks 11 -> 13
Other:
- note added: "row: PD0 column: PD1"
- note removed: "row: PD0 column: PD1 led: PD4"
